File: keyboard.kicad_pcb (KiCad board)
At the start: 2 copper layers, 101 parts, among them U1 ProMicro

Commit message: aligned all components
Parts:
- moved D_SHIFT1 37.5 mm to (307.4, 74.6), turned to 190 degrees
- moved D_B1 18.9 mm to (124.0, 87.7), turned to 170 degrees
- moved D_SHIFT2 17.6 mm to (17.3, 75.4), turned to 170 degrees
- moved D_CTRL1 15.5 mm to (145.3, 106.0), turned to 240 degrees
- moved D_R1 15.5 mm to (112.2, 44.4), turned to 170 degrees
- moved D_ALT1 15.1 mm to (174.7, 106.0), turned to 120 degrees
- moved D_CAPS1 14.8 mm to (25.3, 57.5), turned to 170 degrees
- moved D_ENTER1 14.5 mm to (318.2, 53.4), turned to 190 degrees
- moved D_SUPER1 14.2 mm to (64.8, 94.0), turned to 170 degrees
- moved D_A1 14.1 mm to (51.1, 62.1), turned to 170 degrees
- moved D_ALT2 14.0 mm to (44.5, 99.6), turned to 170 degrees
- moved D_META1 13.9 mm to (84.0, 94.9), turned to 170 degrees
- moved D_N1 13.7 mm to (196.0, 87.7), turned to 190 degrees
- moved D_TAB1 13.5 mm to (30.9, 39.2), turned to 170 degrees
- moved D_Q1 13.4 mm to (54.4, 43.3), turned to 170 degrees
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
Commit message: complete routing
Parts:
- moved K_E1 74.6 mm to (146.2, 55.2)
- moved D_K1 56.6 mm to (280.3, 82.1)
- moved D_COMMA1 56.6 mm to (283.6, 100.9)
- moved D_I1 56.6 mm to (277.0, 63.3)
- moved D_LEFT1 56.6 mm to (286.9, 119.6)
- moved D_O1 56.6 mm to (296.2, 62.5)
- moved D_C1 56.6 mm to (138.2, 100.9)
- moved D_D1 56.6 mm to (141.5, 82.1)
- moved D_E1 56.6 mm to (144.8, 63.3)
- moved D_BKSP1 56.6 mm to (161.6, 131.3)
- moved D_BSLSH1 56.6 mm to (358.7, 60.6)
- moved D_CAPS1 56.6 mm to (76.2, 82.3)
- moved D_CTRL2 56.6 mm to (74.2, 120.6)
- moved D_DOT1 56.6 mm to (302.8, 100.0)
- moved D_DOWN1 56.6 mm to (306.1, 118.8)
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Routing:
- net col9: track 0.00 -> 504.6 mm
- net row3: track 0.00 -> 396.6 mm
- net row2: track 0.00 -> 395.2 mm
- net row1: track 0.00 -> 375.5 mm
- net row0: track 0.00 -> 327.6 mm
- net col12: track 0.00 -> 312.1 mm
- net col11: track 0.00 -> 301.3 mm
- net col10: track 0.00 -> 251.6 mm
- net col8: track 0.00 -> 214.2 mm
- net col0: track 0.00 -> 213.8 mm
- net col1: track 0.00 -> 192.1 mm
- net col2: track 0.00 -> 165.2 mm
- net col3: track 0.00 -> 148.8 mm
- net col7: track 0.00 -> 147.2 mm, vias 0 -> 1
- net col4: track 0.00 -> 137.4 mm
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- removed copper zone on B.Cu, net GND
- removed copper zone on F.Cu, net VCC
Other:
- board outline added: 349.7 x 114.3 mm

Commit message: add reset switch and ground zones
Parts:
- added SW1: SW_PUSH, kbd:ResetSW, F.Cu at (210.9, 93.7)
Connections:
- U1 pad 22: Net-(U1-Pad22) -> RESET
- U1 pad 23: Net-(U1-Pad23) -> GND
- U1 pad 3: Net-(U1-Pad3) -> GND
- U1 pad 4: Net-(U1-Pad4) -> GND
Routing:
- net col9: track 504.6 -> 313.8 mm
- net RESET: track 0.00 -> 32.9 mm
- net col10: track 251.6 -> 249.9 mm
- net col8: track 214.2 -> 212.7 mm
- net col11: track 301.3 -> 300.6 mm
- net row3: track 396.6 -> 396.0 mm
- added copper zone on B.Cu, net GND
- added copper zone on F.Cu, net GND
