File: pcb/keyboard.kicad_pcb (KiCad board)
At the start: 2 copper layers, 349.7 x 114.3 mm, 102 parts, among them SW1 SW_PUSH, U1 ProMicro

Commit message: remove zones and reroute ground
Routing:
- net GND: track 0.00 -> 44.3 mm, vias 0 -> 2
- removed copper zone on B.Cu, net GND
- removed copper zone on F.Cu, net GND
Changed lines of the file:
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@@
     (thickness 1.6)
     (drawings 16)
-    (tracks 869)
+    (tracks 880)
     (zones 0)
     (modules 102)
@@
       (drillshape 0)
       (scaleselection 1)
-      (outputdirectory "Gerber/"))
+      (outputdirectory "gerber/"))
   )
   (net 0 "")
@@
   (segment (start 207.6268 92.311787) (end 206.626801 91.311788) (width 0.25) (layer B.Cu) (net 71))
   (segment (start 206.626801 70.717001) (end 206.626801 82.425199) (width 0.25) (layer B.Cu) (net 71))
-  (zone (net 72) (net_name GND) (layer B.Cu) (hatch edge 0.508)
-    (connect_pads (clearance 0.508))
-    (min_thickness 0.254)
-    (fill yes (arc_segments 32) (thermal_gap 0.508) (thermal_bridge_width 0.508))
-    (polygon
-      (pts
-        (xy 424.18 162.56) (xy 424.18 27.94) (xy 35.56 27.94) (xy 35.56 162.56)
-      )
-    )
-  )
-  (zone (net 72) (net_name GND) (layer F.Cu) (hatch edge 0.508)
-    (connect_pads (clearance 0.508))
-    (min_thickness 0.254)
-    (fill yes (arc_segments 32) (thermal_gap 0.508) (thermal_bridge_width 0.508))
-    (polygon
-      (pts
-        (xy 35.56 162.56) (xy 35.56 27.94) (xy 424.18 27.94) (xy 424.18 162.56)
-      )
-    )
-  )
+  (segment (start 203.2682 64.8184) (end 205.7884 64.8184) (width 0.25) (layer F.Cu) (net 72))
+  (segment (start 205.7884 64.8184) (end 208.28 67.31) (width 0.25) (layer F.Cu) (net 72))
+  (via (at 212.221653 67.441653) (size 0.8) (drill 0.4) (layers F.Cu B.Cu) (net 72))
+  (segment (start 212.304906 67.3584) (end 212.221653 67.441653) (width 0.25) (layer F.Cu) (net 72))
+  (segment (start 218.4882 67.3584) (end 212.304906 67.3584) (width 0.25) (layer F.Cu) (net 72))
+  (segment (start 212.221653 67.441653) (end 208.411653 67.441653) (width 0.25) (layer B.Cu) (net 72))
+  (segment (start 218.4882 69.8984) (end 218.4882 67.3584) (width 0.25) (layer F.Cu) (net 72))
+  (segment (start 214.1268 93.726) (end 215.36996 92.48284) (width 0.25) (layer F.Cu) (net 72))
+  (segment (start 215.36996 73.01664) (end 218.4882 69.8984) (width 0.25) (layer F.Cu) (net 72))
+  (segment (start 215.36996 92.48284) (end 215.36996 73.01664) (width 0.25) (layer F.Cu) (net 72))
+  (via (at 208.411653 67.441653) (size 0.8) (drill 0.4) (layers F.Cu B.Cu) (net 72))
 )

Commit message: clean up routes
Routing:
- net col9: track 313.8 -> 234.8 mm
- net col0: track 213.8 -> 214.6 mm
